Commit message: modified:   champ/champ_bringup/launch/bringup.launch.py 	new file:   robots/descriptions/go2_description/meshes/mid-360-asm.stl 	modified:   robots/descriptions/go2_description/xacro/mid360.xacro 	modified:   robots/descriptions/go2_description/xacro/robot_mid360.xacro

File: robots/descriptions/go2_description/xacro/mid360.xacro (robot description, xacro)
@@ -19,44 +19,35 @@
     </inertial>
   </xacro:macro>
-  <xacro:macro name="mid360" params="name:='' parent:= 'base_link' topic:='mid360' *origin ">
-    <link name="${name}">
+  <xacro:macro name="mid360" params="name:='' parent:= 'base_link' topic:='mid360' downsample:='1' visualize:='true' *origin ">
+    <link name="${name}_frame">
+        <xacro:if value="${visualize}">
         <visual>
-        <origin rpy="0 0 0" xyz="0 0 0"/>
-        <geometry>
-            <sphere radius="0.03"/>
-        </geometry>
-        <material name="lidar_color">
-            <color rgba="1.0 0.4 0.2 1"/>
-        </material>
+            <origin rpy="1.57 0 3.14" xyz="0 0 0"/>
+            <geometry>
+                <mesh filename="file://$(find go2_description)/meshes/mid-360-asm.stl" scale="0.001 0.001 0.001"/>
+            </geometry>
         </visual>
-        <visual>
-        <origin rpy="0 0 0" xyz="0 0 -0.02"/>
-        <geometry>
-            <box size="0.08 0.08 0.04"/>
-        </geometry>
-        <material name="lidar_base_color">
-            <color rgba="0.5 0.5 0.5 0.8"/>
-        </material>
-        </visual>
-        <collision>
-        <origin rpy="0 0 0" xyz="0 0 0"/>
-        <geometry>
-            <sphere radius="0.03"/>
-        </geometry>
-        </collision>
-        <collision>
-        <origin rpy="0 0 0" xyz="0 0 -0.02"/>
-        <geometry>
-            <box size="0.08 0.08 0.04"/>
-        </geometry>
-        </collision>
+        </xacro:if>
+      <collision>
+		  <origin xyz="0 0 0" rpy="1.57 0 3.14" />
+      <geometry>
+         <mesh filename="file://$(find go2_description)/meshes/mid-360-asm.stl" scale="0.001 0.001 0.001"/>
+      </geometry>
+      </collision>
     </link>
     <joint name="${name}_joint" type="fixed">
       <parent link="${parent}"/>
-      <child link="${name}"/>
+      <child link="${name}_frame"/>
       <xacro:insert_block name="origin"/>
     </joint>
-    <gazebo reference="${name}">
-      <sensor type="ray" name="${name}">
+    <link name="${name}_imu_link">
+    </link>
+    <joint name="${name}_imu_joint" type="fixed">
+        <origin rpy="0 0 0" xyz="0.0 0 0"/>
+        <parent link="${name}_frame"/>
+        <child link="${name}_imu_link"/>
+    </joint>
+    <gazebo reference="${name}_frame">
+      <sensor type="ray" name="${name}_frame">
         <pose>0 0 0 0 0 0</pose>
         <visualize>true</visualize>
@@ -92,5 +83,5 @@
           <visualize>false</visualize>
 		  <samples>${samples}</samples>
-		  <downsample>1</downsample>
+		  <downsample>${downsample}</downsample>
 		  <csv_file_name>$(find ros2_livox_simulation)/scan_mode/mid360.csv</csv_file_name>
 		  <topic>${topic}</topic>
@@ -98,4 +89,28 @@
       </sensor>
     </gazebo>
+    <gazebo reference="${name}_imu_link">
+        <gravity>true</gravity>
+        <sensor name="${name}imu_sensor" type="imu">
+        <always_on>true</always_on>
+        <update_rate>100</update_rate>
+        <visualize>true</visualize>
+        <topic>__default_topic__</topic>
+        <pose>0 0 0 0 0 0</pose>
+        <plugin filename="libgazebo_ros_imu_sensor.so" name="${name}_imu_plugin">
+            <ros>
+            <namespace>livox</namespace>
+            <remapping>${name}_imu_plugin/out:=/${name}/imu</remapping>
+            </ros>
+            <topicName>imu</topicName>
+            <bodyName>${name}_imu_link</bodyName>
+            <updateRateHZ>100.0</updateRateHZ>
+            <gaussianNoise>0.0001</gaussianNoise>
+            <xyzOffset>0 0 0</xyzOffset>
+            <rpyOffset>0 0 0</rpyOffset>
+            <frame_name>${name}_imu_link</frame_name>
+            <initial_orientation_as_reference>false</initial_orientation_as_reference>
+        </plugin>
+        </sensor>
+    </gazebo>
   </xacro:macro>
 </robot>

File: robots/descriptions/go2_description/xacro/robot_mid360.xacro (robot description, xacro)
@@ -80,4 +80,34 @@
         </collision>
     </link>
+    <link
+        name="unitree_lidar">
+        <inertial>
+        <origin
+            xyz="0 0 0"
+            rpy="0 0 0" />
+        <mass
+            value="0" />
+        <inertia
+            ixx="0"
+            ixy="0"
+            ixz="0"
+            iyy="0"
+            iyz="0"
+            izz="0" />
+        </inertial>
+    </link>
+    <joint
+        name="radar_joint"
+        type="fixed">
+        <origin
+        xyz="0.28945 0 -0.046825"
+        rpy="0 2.8782 0" />
+        <parent
+        link="trunk" />
+        <child
+        link="unitree_lidar" />
+        <axis
+        xyz="0 0 0" />
+    </joint>
     <!--
     <joint name="load_joint" type="fixed">
@@ -111,6 +141,9 @@
     <xacro:leg name="lh" mirror="1"  mirror_dae="True"   front_hind="-1" front_hind_dae="False" />
     <xacro:include filename="$(find go2_description)/xacro/mid360.xacro"/>
-    <xacro:mid360 name="livox" parent="imu_link" topic="livox/cloud">
+    <xacro:mid360 name="livox" parent="imu_link" topic="livox/lidar">
         <origin xyz="0.1870 0 0.0803" rpy="0 0.2268928 0"/>
+    </xacro:mid360>
+    <xacro:mid360 name="utlidar_lidar" parent="unitree_lidar" topic="utlidar/cloud" downsample='10' visualize="false" >
+        <origin xyz="0 0 0" rpy="0 0 0"/>
     </xacro:mid360>
     <!-- <xacro:include filename="$(find go2_description)/xacro/laser.xacro"/> -->

Commit message: new file:   robots/descriptions/go2_description/meshes/livox_mid360.dae 	deleted:    robots/descriptions/go2_description/meshes/mid-360-asm.stl 	modified:   robots/descriptions/go2_description/xacro/mid360.xacro 	modified:   robots/descriptions/go2_description/xacro/robot_mid360.xacro

File: robots/descriptions/go2_description/xacro/mid360.xacro (robot description, xacro)
@@ -8,31 +8,38 @@
     <xacro:property name="noise_mean" value="0.0"/>
     <xacro:property name="noise_stddev" value="0.01"/>
-    <xacro:property name="mass" value="0.4" />
-    <xacro:property name="length" value="0.05" />
-    <xacro:property name="width" value="0.05" />
-    <xacro:property name="height" value="0.02" />
-  <xacro:macro name="box_inertia" params="m w h d">
-    <inertial>
-      <origin xyz="0 0 0" rpy="${pi/2} 0 ${pi/2}"/>
-      <mass value="${m}"/>
-      <inertia ixx="${(m/12) * (h*h + d*d)}" ixy="0.0" ixz="0.0" iyy="${(m/12) * (w*w + d*d)}" iyz="0.0" izz="${(m/12) * (w*w + h*h)}"/>
-    </inertial>
-  </xacro:macro>
+    <!-- 修正质量参数（Livox Mid360实际重量约220g） -->
+    <xacro:property name="mass" value="0.22" />
+    <xacro:property name="length" value="0.05" />  <!-- X轴方向尺寸 -->
+    <xacro:property name="width" value="0.05" />   <!-- Y轴方向尺寸 -->
+    <xacro:property name="height" value="0.02" />  <!-- Z轴方向尺寸 -->
   <xacro:macro name="mid360" params="name:='' parent:= 'base_link' topic:='mid360' downsample:='1' visualize:='true' *origin ">
     <link name="${name}_frame">
-        <xacro:if value="${visualize}">
+      <xacro:if value="${visualize}">
         <visual>
-            <origin rpy="1.57 0 3.14" xyz="0 0 0"/>
+            <origin rpy="0 0 1.57" xyz="0 0 0"/>
             <geometry>
-                <mesh filename="file://$(find go2_description)/meshes/mid-360-asm.stl" scale="0.001 0.001 0.001"/>
+                <mesh filename="file://$(find go2_description)/meshes/livox_mid360.dae"/>
             </geometry>
         </visual>
-        </xacro:if>
-      <collision>
-		  <origin xyz="0 0 0" rpy="1.57 0 3.14" />
-      <geometry>
-         <mesh filename="file://$(find go2_description)/meshes/mid-360-asm.stl" scale="0.001 0.001 0.001"/>
-      </geometry>
-      </collision>
+        <collision>
+        <origin xyz="0 0 0" rpy="0 0 1.57" />
+            <geometry>
+              <mesh filename="file://$(find go2_description)/meshes/livox_mid360.dae"/>
+            </geometry>
+        </collision>
+        <inertial>
+          <!-- 移除冗余旋转，保持坐标系与link一致 -->
+          <origin xyz="0 0 0" rpy="0 0 0"/>
+          <mass value="${mass}"/>
+          <!-- 修正惯性张量计算公式 -->
+          <inertia
+              ixx="${(mass/12) * (width**2 + height**2)}"
+              ixy="0.0"
+              ixz="0.0"
+              iyy="${(mass/12) * (length**2 + height**2)}"
+              iyz="0.0"
+              izz="${(mass/12) * (length**2 + width**2)}"/>
+        </inertial>
+      </xacro:if>
     </link>
     <joint name="${name}_joint" type="fixed">
@@ -41,4 +48,5 @@
       <xacro:insert_block name="origin"/>
     </joint>
+    <!-- 以下部分保持不变 -->
     <link name="${name}_imu_link">
     </link>
@@ -66,6 +74,6 @@
 				<samples>360</samples>
 				<resolution>1</resolution>
-        <min_angle>${-55.22/180*pi}</min_angle>
-        <max_angle>${7.22/180*pi}</max_angle>
+                <min_angle>${-55.22/180*pi}</min_angle>
+                <max_angle>${7.22/180*pi}</max_angle>
 				</vertical>
 			  </scan>

File: robots/descriptions/go2_description/xacro/robot_mid360.xacro (robot description, xacro)
@@ -141,9 +141,9 @@
     <xacro:leg name="lh" mirror="1"  mirror_dae="True"   front_hind="-1" front_hind_dae="False" />
     <xacro:include filename="$(find go2_description)/xacro/mid360.xacro"/>
-    <xacro:mid360 name="livox" parent="imu_link" topic="livox/lidar">
+    <xacro:mid360 name="livox" parent="imu_link" topic="livox/lidar" downsample='1' visualize="true" >
         <origin xyz="0.1870 0 0.0803" rpy="0 0.2268928 0"/>
     </xacro:mid360>
     <xacro:mid360 name="utlidar_lidar" parent="unitree_lidar" topic="utlidar/cloud" downsample='10' visualize="false" >
-        <origin xyz="0 0 0" rpy="0 0 0"/>
+        <origin xyz="0 0 0.2" rpy="0 0 0"/>
     </xacro:mid360>
     <!-- <xacro:include filename="$(find go2_description)/xacro/laser.xacro"/> -->

Commit message: modified:   robots/descriptions/go2_description/xacro/mid360.xacro 	modified:   robots/descriptions/go2_description/xacro/robot_mid360.xacro

File: robots/descriptions/go2_description/xacro/mid360.xacro (robot description, xacro)
@@ -8,9 +8,8 @@
     <xacro:property name="noise_mean" value="0.0"/>
     <xacro:property name="noise_stddev" value="0.01"/>
-    <!-- 修正质量参数（Livox Mid360实际重量约220g） -->
     <xacro:property name="mass" value="0.22" />
-    <xacro:property name="length" value="0.05" />  <!-- X轴方向尺寸 -->
-    <xacro:property name="width" value="0.05" />   <!-- Y轴方向尺寸 -->
-    <xacro:property name="height" value="0.02" />  <!-- Z轴方向尺寸 -->
+    <xacro:property name="length" value="0.05" />
+    <xacro:property name="width" value="0.05" />
+    <xacro:property name="height" value="0.02" />
   <xacro:macro name="mid360" params="name:='' parent:= 'base_link' topic:='mid360' downsample:='1' visualize:='true' *origin ">
     <link name="${name}_frame">
@@ -29,8 +28,6 @@
         </collision>
         <inertial>
-          <!-- 移除冗余旋转，保持坐标系与link一致 -->
           <origin xyz="0 0 0" rpy="0 0 0"/>
           <mass value="${mass}"/>
-          <!-- 修正惯性张量计算公式 -->
           <inertia
               ixx="${(mass/12) * (width**2 + height**2)}"
@@ -48,5 +45,4 @@
       <xacro:insert_block name="origin"/>
     </joint>
-    <!-- 以下部分保持不变 -->
     <link name="${name}_imu_link">
     </link>

File: robots/descriptions/go2_description/xacro/robot_mid360.xacro (robot description, xacro)
@@ -141,9 +141,9 @@
     <xacro:leg name="lh" mirror="1"  mirror_dae="True"   front_hind="-1" front_hind_dae="False" />
     <xacro:include filename="$(find go2_description)/xacro/mid360.xacro"/>
-    <xacro:mid360 name="livox" parent="imu_link" topic="livox/lidar" downsample='1' visualize="true" >
+    <xacro:mid360 name="livox" parent="imu_link" topic="livox/lidar" downsample='2' visualize="true" >
         <origin xyz="0.1870 0 0.0803" rpy="0 0.2268928 0"/>
     </xacro:mid360>
-    <xacro:mid360 name="utlidar_lidar" parent="unitree_lidar" topic="utlidar/cloud" downsample='10' visualize="false" >
-        <origin xyz="0 0 0.2" rpy="0 0 0"/>
+    <xacro:mid360 name="utlidar_lidar" parent="unitree_lidar" topic="utlidar/cloud" downsample='5' visualize="false" >
+        <origin xyz="0 0 0.1" rpy="0 0 0"/>
     </xacro:mid360>
     <!-- <xacro:include filename="$(find go2_description)/xacro/laser.xacro"/> -->
